File: bmp_4pin_50mil_swd/V1.1/bmp_4pin_50mil_swd.kicad_pcb (KiCad board)
At the start: 2 copper layers, 15.2 x 5.5 mm, 13 parts, among them J1 4Pin_50mil_SWD, X1 JTAG-10

Commit message: Added OSHPark link.
Parts:
- moved REF** 1.00 mm to (30.1, 25.9)
- moved REF** 1.00 mm to (23.6, 25.9)
- moved REF** 1.00 mm to (27.0, 25.9)
- moved REF** 1.00 mm to (20.6, 25.9)
- moved REF** 1.00 mm to (32.6, 25.9)
- moved REF** 0.87 mm to (20.8, 23.6)
- moved J1 0.50 mm to (34.1, 23.2)
- moved LOGO1 0.50 mm to (21.6, 22.9)
- moved LOGO2 0.50 mm to (21.6, 22.9)
- moved X1 0.50 mm to (26.4, 23.2)
Other:
- board size 15.2 x 5.5 mm -> 15.2 x 6.5 mm
